File: Eagle/LED MATRIX PTH.sch (EAGLE design)
At the start: 19 parts, among them J1 2013499-1, J2 AVR_SPI_PROG_3X2NS, U2 328P, Y1 16MHz

Commit message: Added Gerbers and modified schematic
Parts:
- removed C3: 1uF, resistor:CPOL-EUSMCA
- removed C5: 10uF, SparkFun-Capacitors:10UF-POLAR-EIA3216-16V-10%(TANT)
- removed D66: (no value), SparkFun-LED:LED0603
- removed IC7805: (no value), SparkFun-IC-Power:V_REG_78XX-TO-220
- removed R10: 330, SparkFun-Resistors:330OHM-0603-1/10W-1%
- removed SV1: (no value), con-lstb:MA06-1
- removed SV2: (no value), con-lstb:MA07-2
- added D10, D11, D12, D13, D14, D15, D16, D17, D18, D19, D2, D20, D21, D22, D23, D24, D25, D26, D27, D28, D29, D3, D30, D31, D32, D33, D34, D35, D36, D37, D38, D39, D4, D40, D41, D42, D43, D44, D45, D46, D47, D48, D49, D5, D50, D51, D52, D53, D54, D55, D56, D57, D58, D59, D6, D60, D61, D62, D63, D64, D7, D8, D9: (no value), SparkFun-LED:LED5MM
- added D65: BLUE, SparkFun-LED:LED-BLUE0603
- added R3, R4, R5, R6, R7, R8: 10k, SparkFun-Resistors:10KOHM-0603-1/10W-1%
- added R9: 330, SparkFun-Resistors:330OHM-0603-1/10W-1%
- added S2, S3, S4, S5, S6, S7: 2-1437565-7, 2-1437565-7:2-1437565-7
- added U1: 328P, SparkFun-IC-Microcontroller:ATMEGA328P_PDIP
- added U3: (no value), SparkFun-IC-Power:V_REG_78XXSIDE
- D1: device SparkFun-LED:LED0603 -> SparkFun-LED:LED5MM
- J1: value 2013499-1 -> AVR_SPI_PROG_3X2NS; device 2013499-1:2013499-1 -> SparkFun-Connectors:AVR_SPI_PROG_3X2NS
- J2: value AVR_SPI_PROG_3X2NS -> 2013499-1; device SparkFun-Connectors:AVR_SPI_PROG_3X2NS -> 2013499-1:2013499-1
- R2: value 330 -> 22k; device SparkFun-Resistors:330OHM-0603-1/10W-1% -> SparkFun-Resistors:22KOHM-0603-1/10W-1%
- S1: value (none) -> 2-1437565-7; device SparkFun:TAC_SWITCHSMD -> 2-1437565-7:2-1437565-7
- U$1: value 2MMS_SLIDE_SWITCH -> TS02_SWITCH; device 2MMS_SLIDE_SWITCH:2MMS_SLIDE_SWITCH -> 2.54mm slide switch:TS02_SWITCH
- U2: value 328P -> MAX7219CWGT; device SparkFun-IC-Microcontroller:ATMEGA328P_PDIP -> MAX7219CWGT:MAX7219CWGT
Connections:
- removed net 5VBAT: C5.+, IC7805.OUT, U$1.PIN3
- removed net 5VUSB: J1.VBUS, U$1.PIN1
- removed net A0: SV1.1, U2.PC0(ADC0)
- removed net A1: SV1.2, U2.PC1(ADC1)
- removed net A2: SV1.3, U2.PC2(ADC2)
- removed net A3: SV1.4, U2.PC3(ADC3)
- removed net A4: SV1.5, U2.PC4(ADC4/SDA)
- removed net A5: SV1.6, U2.PC5(ADC5/SCL)
- removed net DIGITAL_PIN_0: SV2.1, U2.PD0(RXD)
- removed net DIGITAL_PIN_1: SV2.2, U2.PD1(TXD)
- removed net DIGITAL_PIN_10: SV2.11, U2.PB2(SS/OC1B)
- removed net DIGITAL_PIN_2: SV2.3, U2.PD2(INT0)
- removed net DIGITAL_PIN_3: SV2.4, U2.PD3(INT1)
- removed net DIGITAL_PIN_4: SV2.5, U2.PD4(XCK/T0)
- removed net DIGITAL_PIN_5: SV2.6, U2.PD5(T1)
- removed net DIGITAL_PIN_6: SV2.7, U2.PD6(AIN0)
- removed net DIGITAL_PIN_7: SV2.8, U2.PD7(AIN1)
- removed net DIGITAL_PIN_8: SV2.9, U2.PB0(ICP)
- removed net DIGITAL_PIN_9: SV2.10, U2.PB1(OC1A)
- removed net MISO(DIGITAL_PIN_12): J2.1, SV2.13, U2.PB4(MISO)
- removed net MOSI(DIGITAL_PIN_11): J2.4, SV2.12, U2.PB3(MOSI/OC2)
- removed net N$5: D66.C, R10.2
- removed net N$7: D1.C, R2.2
- removed net SCK(DIGITAL_PIN_13): D66.A, J2.3, SV2.14, U2.PB5(SCK)
- new net +5V: D65.A, J1.2, R1.2, S2.1, S2.2, S3.1, S3.2, S4.1, S4.2, S5.1, S5.2, S6.1, S6.2, S7.1, S7.2, U1.AVCC, U1.VCC
- new net 5V_BAT: U$1.PIN3, U3.OUT
- new net 5V_USB: J2.VBUS, U$1.PIN1
- new net C0: D1.A, D10.A, D11.A, D12.A, D13.A, D14.A, D15.A, D9.A, U2.DIG_0
- new net C1: D16.A, D17.A, D18.A, D19.A, D2.A, D20.A, D21.A, D22.A, U2.DIG_1
- new net C2: D23.A, D24.A, D25.A, D26.A, D27.A, D28.A, D29.A, D3.A, U2.DIG_2
- new net C3: D30.A, D31.A, D32.A, D33.A, D34.A, D35.A, D36.A, D4.A, U2.DIG_3
- new net C4: D37.A, D38.A, D39.A, D40.A, D41.A, D42.A, D43.A, D5.A, U2.DIG_4
- new net C5: D44.A, D45.A, D46.A, D47.A, D48.A, D49.A, D50.A, D6.A, U2.DIG_5
- new net C6: D51.A, D52.A, D53.A, D54.A, D55.A, D56.A, D57.A, D7.A, U2.DIG_6
- new net C7: D58.A, D59.A, D60.A, D61.A, D62.A, D63.A, D64.A, D8.A, U2.DIG_7
- new net CLK: U1.PB2(SS/OC1B), U2.CLK
- new net DIN: U1.PB0(ICP), U2.DIN
- new net DOUT: U2.DOUT
- new net DOWN: R4.1, S3.3, S3.4, U1.PC1(ADC1)
- new net LEFT: R5.1, S4.3, S4.4, U1.PC2(ADC2)
- new net LOAD: U1.PB1(OC1A), U2.LOAD
- new net MISO: J1.1, U1.PB4(MISO)
- new net MOSI: J1.4, U1.PB3(MOSI/OC2)
- new net N$4: D65.C, R9.2
- new net OK: R7.1, S6.3, S6.4, U1.PC4(ADC4/SDA)
- new net R0: D1.C, D2.C, D3.C, D4.C, D5.C, D6.C, D7.C, D8.C, U2.SEG_DP
- new net R1: D16.C, D23.C, D30.C, D37.C, D44.C, D51.C, D58.C, D9.C, U2.SEG_A
- new net R2: D10.C, D17.C, D24.C, D31.C, D38.C, D45.C, D52.C, D59.C, U2.SEG_B
- new net R3: D11.C, D18.C, D25.C, D32.C, D39.C, D46.C, D53.C, D60.C, U2.SEG_C
- new net R4: D12.C, D19.C, D26.C, D33.C, D40.C, D47.C, D54.C, D61.C, U2.SEG_D
- new net R5: D13.C, D20.C, D27.C, D34.C, D41.C, D48.C, D55.C, D62.C, U2.SEG_E
- new net R6: D14.C, D21.C, D28.C, D35.C, D42.C, D49.C, D56.C, D63.C, U2.SEG_F
- new net R7: D15.C, D22.C, D29.C, D36.C, D43.C, D50.C, D57.C, D64.C, U2.SEG_G
- new net REST: R8.1, S7.3, S7.4, U1.PC5(ADC5/SCL)
- new net RIGHT: R6.1, S5.3, S5.4, U1.PC3(ADC3)
- new net SCK: J1.3, U1.PB5(SCK)
- new net UP: R3.1, S2.3, S2.4, U1.PC0(ADC0)
- new net V_BAT: J3.1, U3.IN
- net 5V: now also R2.2, U2.V+; no longer D1.A, J2.2, R1.2, U2.AVCC, U2.VCC
- net GND: now also J1.6, J2.GND, J3.2, R3.2, R4.2, R5.2, R6.2, R7.2, R8.2, R9.1, U1.GND, U2.GND_2, U3.GND; no longer C3.-, C5.-, IC7805.GND, J1.GND, J2.6, J3.1, R10.1, R2.1
- net N$1: now also C2.2, U1.PB7(XTAL2/TOSC2), Y1.1; no longer C1.2, U2.PB6(XTAL1/TOSC1), Y1.2
- net N$2: now also C1.2, U1.PB6(XTAL1/TOSC1), Y1.2; no longer C2.2, U2.PB7(XTAL2/TOSC2), Y1.1
- net N$3: now also R2.1, U2.ISET; no longer C3.+, IC7805.IN, J3.2
- net RESET: now also J1.5, U1.PC6(/RESET); no longer J2.5, U2.PC6(/RESET)
Other:
- note added: "ISP INTERFACE"
- note added: "JP_PWR"
- note added: "LED_MATRIX"
- note added: "MATRIX_DRIVER"
- note added: "MCU"
- note added: "OP_SWITCHES"
- note added: "PWR_LED"
- note added: "PWR_SW"
- note added: "PWR_USB"
- note added: "REG_5V"
- note removed: "10-12-2019"
- note removed: "5V Regulator"
- note removed: "ATmega328P"
- note removed: "ATmega328P Minimal Ckt"
- note removed: "Analog Pins"
- note removed: "Builtin"
- note removed: "Connections"
- note removed: "DESIGNER: Pranav Srinivas"
- note removed: "Digital Pins"
- note removed: "ISP Programmer"
- note removed: "LED_Uno"
- note removed: "MINIMAL CIRCUIT OF ATMEGA328P"
- note removed: "PWR LED"
- note removed: "SWITCH"
- note removed: "USB Supply"
- note removed: "to"
- moved on the sheet: C1, C2, J3, R1, R2, Y1
